File: ESPLock PCB/ESPLock.kicad_pcb (KiCad board)
At the start: 2 copper layers, 94 x 47 mm, 15 parts, among them J1 servo, J2 RC522, J3 button, J4 Neopixel, J5 Conn_01x15_Pin, J6 Conn_01x15_Pin, J7 voltage input, U1 L7805

Commit message: Add files via upload
Parts:
- added SW1: ~, Omikron:microswitch, F.Cu at (184.0, 81.5)
- moved J3 5.00 mm to (182.0, 75.0)
- moved C2 2.00 mm to (112.0, 65.0)
- moved C3 2.00 mm to (112.0, 55.5)
Routing:
- net Net-(ESP32-Devkit-V1-Omikron1-D4_4): track 30.1 -> 37.8 mm
- net VCC: track 19.1 -> 21.1 mm
- net Net-(D1-A): track 119.9 -> 121.9 mm
- net GND: track 141.5 -> 139.9 mm
- net Net-(ESP32-Devkit-V1-Omikron1-3V3): track 67.0 -> 68.1 mm
Other:
- board text added: "In 7-12V"
- board text added: "github.com/BrychtaJan/ESPLock"
