File: ESPLock PCB/ESPLock.kicad_sch (KiCad schematic)
At the start: 15 parts, among them J1 servo, J2 RC522, J3 button, J4 Neopixel, J5 Conn_01x15_Pin, J6 Conn_01x15_Pin, J7 voltage input, U1 L7805

Commit message: Add files via upload
Parts:
- added microswitch1: ~, Omikron:microswitch, symbol Omikron:microswitch
Connections:
- net at ESP32-Devkit-V1-Omikron1.20 (D4_4), J3.2 (Pin_2), J6.5 (Pin_5)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: now also microswitch1.2
- net at C1.1, ESP32-Devkit-V1-Omikron1.16 (3V3), J2.1 (Pin_1)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: now also microswitch1.4
Changed lines of the file:
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@@
+	)
+	(junction
+		(at 180.34 26.67)
+		(diameter 0)
+		(color 0 0 0 0)
 	)
 	(junction
@@
 	)
 	(junction
+		(at 182.88 30.48)
+		(diameter 0)
+		(color 0 0 0 0)
+	)
+	(junction
 		(at 113.03 96.52)
 		(diameter 0)
@@
 	(wire
 		(pts
+			(xy 180.34 26.67) (xy 180.34 27.94)
+		)
+		(stroke
+			(width 0)
+			(type default)
+		)
+	)
+	(wire
+		(pts
 			(xy 77.47 64.77) (xy 92.71 64.77)
 		)
@@
 	(wire
 		(pts
+			(xy 182.88 30.48) (xy 182.88 74.93)
+		)
+		(stroke
+			(width 0)
+			(type default)
+		)
+	)
+	(wire
+		(pts
 			(xy 149.86 74.93) (xy 162.56 74.93)
 		)
@@
 	(wire
 		(pts
+			(xy 180.34 26.67) (xy 200.66 26.67)
+		)
+		(stroke
+			(width 0)
+			(type default)
+		)
+	)
+	(wire
+		(pts
 			(xy 115.57 96.52) (xy 115.57 90.17)
 		)
@@
 	(wire
 		(pts
-			(xy 180.34 24.13) (xy 180.34 27.94)
+			(xy 180.34 24.13) (xy 180.34 26.67)
 		)
 		(stroke
@@
 	(wire
 		(pts
+			(xy 182.88 30.48) (xy 200.66 30.48)
+		)
+		(stroke
+			(width 0)
+			(type default)
+		)
+	)
+	(wire
+		(pts
 			(xy 177.8 27.94) (xy 180.34 27.94)
 		)
@@
 	(wire
 		(pts
-			(xy 182.88 24.13) (xy 182.88 74.93)
+			(xy 182.88 24.13) (xy 182.88 30.48)
 		)
 		(stroke
@@
 					(unit 1)
 				)
+			)
+		)
+	)
+	(symbol
+		(lib_id "Omikron:microswitch")
+		(at 205.74 29.21 90)
+		(unit 1)
+		(exclude_from_sim no)
+		(in_bom yes)
+		(on_board yes)
+		(dnp no)
+		(fields_autoplaced yes)
+		(property "Reference" "microswitch1"
+			(at 206.375 22.86 90)
+			(effects
+				(font
+					(size 0.381 0.381)
+				)
+			)
+		)
+		(property "Value" "~"
+			(at 206.375 24.13 90)
+			(effects
+				(font
+					(size 1.27 1.27)
+				)
+			)
+		)
+		(property "Footprint" "Omikron:microswitch"
+			(at 195.072 28.702 0)
+			(effects
+				(font
+					(size 1.27 1.27)
+				)
+				(hide yes)
+			)
+		)
+		(property "Datasheet" ""
+			(at 205.74 29.21 0)
+			(effects
+				(font
+					(size 1.27 1.27)
+				)
+				(hide yes)
+			)
+		)
+		(property "Description" ""
+			(at 205.74 29.21 0)
+			(effects
+				(font
+					(size 1.27 1.27)
+				)
+				(hide yes)
+			)
+		)
+		(pin "2"
+		)
+		(pin "1"
+		)
+		(pin "3"
+		)
+		(pin "4"
+		)
+		(instances
+			(project ""
+				(path "/31d5f2dd-d1a9-4f90-8c1c-e9767ed183a0"
+					(reference "microswitch1")
+					(unit 1)
+				)
